File: solartap_mcu_clear.kicad_sch (KiCad schematic)
At the start: 24 parts, among them J1 USB_C_Receptacle_USB2.0_16P, U1 nRF52832-QFxx, U2 RS3002-3.3SYF5

Commit message: Продовая версия без fiducials
Parts:
- removed U2: RS3002-3.3SYF5, Package_TO_SOT_SMD:SOT-23-3, symbol Regulator_Linear:LT1963AxST-3.3
- added C1, C2: 12p, Capacitor_SMD:C_0805_2012Metric_Pad1.18x1.45mm_HandSolder, symbol Device:C_Small
- added U2: RS3002-3.3SYF5, Package_TO_SOT_SMD:SOT-23-5, symbol Regulator_Linear:TLV71209_SOT23-5
- added Y1: 32Mhz, Crystal:Crystal_SMD_3225-4Pin_3.2x2.5mm_HandSoldering, symbol Device:Crystal_GND23_Small
- BT1: value CR2032 -> CR927; footprint Battery:BatteryHolder_MPD_BC2003_1x2032 -> Battery:CR927
- renumbered C11 to C10, C13 to C11, C6 to C3, C5 to C4, C4 to C5, C3 to C6, C2 to C7, C1 to C8, C10 to C9, TP3 to TP1, TP1 to TP3, TP6 to TP4
Connections:
- net GND: now also C1.2, C2.2, U2.2 (GND), Y1.2, Y1.4
- net at C11.1, D2.2 (A): now also U2.5 (OUT)
- net at C12.1, J1.A4 (VBUS), J1.A9 (VBUS)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: now also U2.1 (IN), U2.3 (EN)
- net at U1.34 (XC1): now also C1.1, Y1.1
- net at U1.35 (XC2): now also C2.1, Y1.3
- no-connect marks 39 -> 37
Other:
- note added: "0.9 reg output"
- note added: "1.3 output from LDO"
- note added: "22 pF for 10 turns 61*61 mm w=1 mm, gap=0.4 mm"
- note added: "3.3 supply"
